Commit message: Update battery.urdf.xacro

File: interbotix_ros_xslocobots/interbotix_xslocobot_descriptions/urdf/idm_version/battery.urdf.xacro (robot description, xacro)
@@ -0,0 +1,57 @@
+<?xml version="1.0" ?>
+<robot xmlns:xacro="http://ros.org/wiki/xacro">
+  <xacro:macro name="battery" params="*origin">
+    <joint name="battery" type="fixed">
+      <xacro:insert_block name="origin"/>
+      <parent
+        link="${robot_name}/plate_link"/>
+      <child
+        link="${robot_name}/battery_link"/>
+    </joint>
+    <link name="${robot_name}/battery_link">
+      <visual>
+        <origin
+          rpy="0 0 0"
+          xyz="0 0 0"/>
+        <geometry>
+          <mesh
+            filename="package://interbotix_xslocobot_descriptions/meshes/locobot_meshes/locobot_battery.stl"
+            scale="0.001 0.001 0.001"/>
+        </geometry>
+        <material name="">
+          <color
+            rgba="0.5 0.5 0.5 1"/>
+        </material>
+      </visual>
+      <collision>
+        <origin
+          rpy="0 0 0"
+          xyz="0 0 0"/>
+        <geometry>
+          <mesh
+            filename="package://interbotix_xslocobot_descriptions/meshes/locobot_meshes/locobot_battery.stl"
+            scale="0.001 0.001 0.001"/>
+        </geometry>
+      </collision>
+      <inertial>
+        <origin
+          rpy="0 0 0"
+          xyz="0 0 0.016"/>
+        <mass value="1.194"/>
+        <inertia
+          ixx="0.004312"
+          ixy="0"
+          ixz="0"
+          iyy="0.001908"
+          iyz="0"
+          izz="0.006017"/>
+      </inertial>
+    </link>
+    <gazebo reference="${robot_name}/battery_link">
+      <material>Gazebo/Grey</material>
+    </gazebo>
+    <gazebo reference="battery">
+      <disableFixedJointLumping>true</disableFixedJointLumping>
+    </gazebo>
+  </xacro:macro>
+</robot>
