Commit message: Update arm_cradle.urdf.xacro

File: interbotix_ros_xslocobots/interbotix_xslocobot_descriptions/urdf/idm_version/arm_cradle.urdf.xacro (robot description, xacro)
@@ -2,48 +2,48 @@
 <robot xmlns:xacro="http://ros.org/wiki/xacro">
   <xacro:macro name="arm_cradle" params="*origin">
-    <xacro:if value="${arm_type == 'mobile_wx200'}">
-      <joint name="arm_cradle" type="fixed">
-         <axis xyz="0 0 0"/>
-         <xacro:insert_block name="origin"/>
-         <parent
-          link="${robot_name}/camera_tower_link"/>
-         <child
-          link="${robot_name}/arm_cradle_link"/>
-      </joint>
-     <link name="${robot_name}/arm_cradle_link">
-       <visual>
-         <origin
-          rpy="0 0 0"
-          xyz="0 0 0"/>
-         <geometry>
-           <mesh
-            filename="package://interbotix_xslocobot_descriptions/meshes/locobot_meshes/idm_version/locobot_arm_cradle.stl"
-            scale="${mesh_scale}"/>
-         </geometry>
-         <material name="interbotix_black"/>
-       </visual>
-       <collision>
-         <origin rpy="0 0 0" xyz="0 0 0"/>
-         <geometry>
-           <mesh
-            filename="package://interbotix_xslocobot_descriptions/meshes/locobot_meshes/idm_version/locobot_arm_cradle.stl"
-            scale="${mesh_scale}"/>
-         </geometry>
-       </collision>
-       <inertial>
-         <origin
-          rpy="0 0 0"
-          xyz="0.0014389900 0 0.0098387400"/>
-         <mass value="0.017626"/>
-         <inertia
-          ixx="0.0000046575"
-          ixy="0"
-          ixz="0.0000000748"
-          iyy="0.0000018629"
-          iyz="0"
-          izz="0.0000046198"/>
-       </inertial>
-     </link>
-    </xacro:if>
+    <joint name="arm_cradle" type="fixed">
+       <axis xyz="0 0 0"/>
+       <xacro:insert_block name="origin"/>
+       <parent
+        link="${robot_name}/camera_tower_link"/>
+       <child
+        link="${robot_name}/arm_cradle_link"/>
+    </joint>
+   <link name="${robot_name}/arm_cradle_link">
+     <visual>
+       <origin
+        rpy="0 0 ${pi/2}"
+        xyz="0 0 0"/>
+       <geometry>
+         <mesh
+          filename="package://interbotix_xslocobot_descriptions/meshes/locobot_meshes/idm_version/locobot_arm_cradle.stl"
+          scale="${mesh_scale}"/>
+       </geometry>
+       <material name="interbotix_black"/>
+     </visual>
+     <collision>
+       <origin
+        rpy="0 0 ${pi/2}"
+        xyz="0 0 0"/>
+       <geometry>
+         <mesh
+          filename="package://interbotix_xslocobot_descriptions/meshes/locobot_meshes/idm_version/locobot_arm_cradle.stl"
+          scale="${mesh_scale}"/>
+       </geometry>
+     </collision>
+     <inertial>
+       <origin
+        rpy="0 0 0"
+        xyz="0.0014389900 0 0.0098387400"/>
+       <mass value="0.017626"/>
+       <inertia
+        ixx="0.0000046575"
+        ixy="0"
+        ixz="0.0000000748"
+        iyy="0.0000018629"
+        iyz="0"
+        izz="0.0000046198"/>
+     </inertial>
+   </link>
     <gazebo reference="arm_cradle">
       <disableFixedJointLumping>true</disableFixedJointLumping>
