Commit message: Update pan_and_tilt.urdf.xacro

File: interbotix_ros_xslocobots/interbotix_xslocobot_descriptions/urdf/idm_version/pan_and_tilt.urdf.xacro (robot description, xacro)
@@ -9,4 +9,7 @@
         upper="${pi/2}"
         velocity="${pi}"/>
+      <origin
+        rpy="0 0 0"
+        xyz="0.03 0 0.45"/>
       <xacro:insert_block name="origin"/>
       <parent
