Commit message: Update lidar.urdf.xacro

File: interbotix_ros_xslocobots/interbotix_xslocobot_descriptions/urdf/idm_version/lidar.urdf.xacro (robot description, xacro)
@@ -3,4 +3,7 @@
   <xacro:macro name="lidar" params="*origin">
     <joint name="lidar_tower" type="fixed">
+      <origin
+        rpy="0 0 0"
+        xyz="0 0 0.45"/>
       <xacro:insert_block name="origin"/>
       <parent
@@ -13,5 +16,5 @@
         <origin
           rpy="0 0 0"
-          xyz="0 0 0"/>
+          xyz="-0.08 0 0"/>
         <geometry>
           <mesh
@@ -24,5 +27,5 @@
         <origin
           rpy="0 0 0"
-          xyz="0 0 0"/>
+          xyz="-0.08 0 0"/>
         <geometry>
           <mesh
@@ -48,5 +51,5 @@
       <origin
         rpy="0 0 0"
-        xyz="0 0 0.09425"/>
+        xyz="-0.005 0 0.1"/>
       <parent
         link="${robot_name}/lidar_tower_link"/>
@@ -58,5 +61,5 @@
         <origin
           rpy="0 0 0"
-          xyz="0 0 0"/>
+          xyz="0 0 -0.05"/>
         <geometry>
           <mesh
@@ -69,5 +72,5 @@
         <origin
           rpy="0 0 0"
-          xyz="0 0 -0.0091"/>
+          xyz="0 0 0"/>
         <geometry>
           <cylinder
