Commit message: Update locobot.urdf.xacro

File: interbotix_ros_xslocobots/interbotix_xslocobot_descriptions/urdf/locobot.urdf.xacro (robot description, xacro)
@@ -115,4 +115,11 @@
       </xacro:if> <!-- base_type == 'create3' -->
     </xacro:if> <!-- arm_type == 'mobile_wx200' -->
+    <xacro:if value="${arm_type == 'mobile_rx200'}">
+      <xacro:arm_cradle>
+        <origin
+          rpy="0 0 0"
+          xyz="0.0335 0 0.125"/>
+      </xacro:arm_cradle>
+    </xacro:if> <!-- arm_type == 'mobile_rx200' -->
   </xacro:if> <!-- arm_type != 'mobile_base' -->
   <!-- ********************************** Battery **********************************  -->
