Commit message: Update locobot_rx200.srdf.xacro

File: interbotix_ros_xslocobots/interbotix_xslocobot_moveit/config/srdf/locobot_rx200.srdf.xacro (robot description, xacro)
@@ -43,5 +43,5 @@
     <group_state name="Sleep" group="interbotix_arm">
         <joint name="elbow" value="1.61" />
-        <joint name="shoulder" value="-1.78" />
+        <joint name="shoulder" value="-0.78" />
         <joint name="waist" value="0" />
         <joint name="wrist_angle" value="0.0" />
